Commit message: U shaped robot to practice relative and absolute coordinates

File: body.urdf (robot description, URDF)
Before this commit: robot robot, 2 links, 1 joints
Links:
- added link Link2, mass 1; collision box size=1 1 1; visual box size=1 1 1
- added link Link3, mass 1; collision box size=1 1 1; visual box size=1 1 1
- added link Link4, mass 1; collision box size=1 1 1; visual box size=1 1 1
- added link Link5, mass 1; collision box size=1 1 1; visual box size=1 1 1
- added link Link6, mass 1; collision box size=1 1 1; visual box size=1 1 1
Joints:
- added joint Link1_Link2: type revolute, parent Link1, child Link2, origin xyz=0 0 1 rpy=0 0 0, axis 0 1 0, limit lower=-3.14159 upper=3.14159 effort=0.0 velocity=0.0
- added joint Link2_Link3: type revolute, parent Link2, child Link3, origin xyz=0 0.5 0.5 rpy=0 0 0, axis 0 1 0, limit lower=-3.14159 upper=3.14159 effort=0.0 velocity=0.0
- added joint Link3_Link4: type revolute, parent Link3, child Link4, origin xyz=0 1 0 rpy=0 0 0, axis 0 1 0, limit lower=-3.14159 upper=3.14159 effort=0.0 velocity=0.0
- added joint Link4_Link5: type revolute, parent Link4, child Link5, origin xyz=0 0.5 -0.5 rpy=0 0 0, axis 0 1 0, limit lower=-3.14159 upper=3.14159 effort=0.0 velocity=0.0
- added joint Link5_Link6: type revolute, parent Link5, child Link6, origin xyz=0 0 -1 rpy=0 0 0, axis 0 1 0, limit lower=-3.14159 upper=3.14159 effort=0.0 velocity=0.0
- joint Link0_Link1: origin xyz=0.5 0 1 rpy=0 0 0 -> xyz=0 0 1 rpy=0 0 0
